File: testing/testing.kicad_sch (KiCad schematic)
At the start: 9 parts

Commit message: Testing commit 6
Parts:
- removed D7, D8, D9: LED, symbol Device:LED

Commit message: Testing Commit 7 + Re-enabled things + Other minor naming things
Parts:
- added D7, D8, D9: LED, symbol Device:LED
Connections:
- net +BATT: now also D7.2 (A), D8.2 (A), D9.2 (A)
- net GND: now also D7.1 (K), D8.1 (K), D9.1 (K)

Commit message: Testing Commit 9
Parts:
- removed D4, D5, D6, D7, D8, D9: LED, symbol Device:LED

Commit message: Test Commit 14
Parts:
- added D4, D5, D6: LED, symbol Device:LED
Connections:
- net +BATT: now also D4.2 (A), D5.2 (A), D6.2 (A)
- net GND: now also D4.1 (K), D5.1 (K), D6.1 (K)
