File: testing/testing.kicad_pcb (KiCad board)
At the start: 2 copper layers, 0 parts

Commit message: Testing commit 2
Routing:
- added copper zone on B.Cu, net (none)
Other:
- board outline added: 45.8 x 63.6 mm
Changed lines of the file:
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@@
 	)
 	(net 0 "")
-	(gr_line
-		(start 132.85 66.45)
-		(end 132.85 107.25)
+	(gr_rect
+		(start 121.9 66.55)
+		(end 167.75 130.15)
 		(stroke
-			(width 0.2)
+			(width 0.05)
 			(type default)
 		)
-		(layer "F.Cu")
+		(fill no)
+		(layer "Edge.Cuts")
 	)
-	(gr_line
-		(start 234 107.25)
-		(end 234 60.8)
-		(stroke
-			(width 0.2)
-			(type default)
+	(zone
+		(net 0)
+		(net_name "")
+		(layer "B.Cu")
+		(hatch edge 0.5)
+		(connect_pads
+			(clearance 0.5)
 		)
-		(layer "F.Cu")
-	)
-	(gr_line
-		(start 234 60.8)
-		(end 132.85 60.8)
-		(stroke
-			(width 0.2)
-			(type default)
+		(min_thickness 0.25)
+		(filled_areas_thickness no)
+		(fill yes
+			(thermal_gap 0.5)
+			(thermal_bridge_width 0.5)
+			(island_removal_mode 1)
+			(island_area_min 10)
 		)
-		(layer "F.Cu")
-	)
-	(gr_line
-		(start 132.85 107.25)
-		(end 234 107.25)
-		(stroke
-			(width 0.2)
-			(type default)
+		(polygon
+			(pts
+				(xy 121.9 66.55) (xy 121.9 130.15) (xy 167.75 130.15) (xy 167.75 66.55)
+			)
 		)
-		(layer "F.Cu")
 	)
 	(embedded_fonts no)

Commit message: Testing changes commit 2
Changed lines of the file:
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@@
 	)
 	(net 0 "")
+	(gr_line
+		(start 159.0675 121.285)
+		(end 146.685 121.285)
+		(stroke
+			(width 0.2)
+			(type default)
+		)
+		(layer "F.Cu")
+	)
+	(gr_line
+		(start 135.255 112.395)
+		(end 156.21 116.84)
+		(stroke
+			(width 0.2)
+			(type default)
+		)
+		(layer "F.Cu")
+	)
+	(gr_line
+		(start 146.685 121.285)
+		(end 142.24 124.46)
+		(stroke
+			(width 0.2)
+			(type default)
+		)
+		(layer "F.Cu")
+	)
+	(gr_line
+		(start 154.305 96.52)
+		(end 146.05 93.345)
+		(stroke
+			(width 0.2)
+			(type default)
+		)
+		(layer "F.Cu")
+	)
+	(gr_line
+		(start 161.925 100.965)
+		(end 159.0675 121.285)
+		(stroke
+			(width 0.2)
+			(type default)
+		)
+		(layer "F.Cu")
+	)
+	(gr_line
+		(start 146.05 93.345)
+		(end 135.255 112.395)
+		(stroke
+			(width 0.2)
+			(type default)
+		)
+		(layer "F.Cu")
+	)
+	(gr_line
+		(start 156.21 116.84)
+		(end 161.925 100.965)
+		(stroke
+			(width 0.2)
+			(type default)
+		)
+		(layer "F.Cu")
+	)
+	(gr_line
+		(start 142.24 124.46)
+		(end 154.305 96.52)
+		(stroke
+			(width 0.2)
+			(type default)
+		)
+		(layer "F.Cu")
+	)
 	(gr_rect
 		(start 121.9 66.55)

Commit message: testing diff_changes v2
Parts:
- added REF**: BatteryClip_Keystone_54_D16-19mm, Battery:BatteryClip_Keystone_54_D16-19mm, F.Cu at (127.0, 118.7)
Routing:
- net (no net): vias 0 -> 8

Commit message: Merge Workflows + Test
Parts:
- removed REF**: BatteryClip_Keystone_54_D16-19mm, Battery:BatteryClip_Keystone_54_D16-19mm

Commit message: Testing commit 3
Routing:
- net (no net): vias 8 -> 15
Changed lines of the file:
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@@
+	)
+	(via
+		(at 153.035 76.2)
+		(size 0.6)
+		(drill 0.3)
+		(layers "F.Cu" "B.Cu")
+		(net 0)
 	)
 	(via
@@
 	)
 	(via
+		(at 147.955 78.74)
+		(size 0.6)
+		(drill 0.3)
+		(layers "F.Cu" "B.Cu")
+		(net 0)
+	)
+	(via
+		(at 146.05 71.12)
+		(size 0.6)
+		(drill 0.3)
+		(layers "F.Cu" "B.Cu")
+		(net 0)
+	)
+	(via
 		(at 153.67 88.265)
+		(size 0.6)
+		(drill 0.3)
+		(layers "F.Cu" "B.Cu")
+		(net 0)
+	)
+	(via
+		(at 153.035 83.82)
 		(size 0.6)
 		(drill 0.3)
@@
 		(size 0.6)
 		(drill 0.3)
+		(layers "F.Cu" "B.Cu")
+		(net 0)
+	)
+	(via
+		(at 130.175 85.09)
+		(size 0.6)
+		(drill 0.3)
+		(layers "F.Cu" "B.Cu")
+		(net 0)
+	)
+	(via
+		(at 146.05 84.455)
+		(size 0.6)
+		(drill 0.3)
+		(layers "F.Cu" "B.Cu")
+		(net 0)
+	)
+	(via
+		(at 133.35 79.375)
+		(size 0.6)
+		(drill 0.3)

Commit message: Testing commit 4
Routing:
- net (no net): vias 15 -> 10
Changed lines of the file:
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@@
-	)
-	(via
-		(at 132.08 93.98)
-		(size 0.6)
-		(drill 0.3)
-		(layers "F.Cu" "B.Cu")
-		(net 0)
 	)
 	(via
@@
 	)
 	(via
-		(at 133.985 83.82)
-		(size 0.6)
-		(drill 0.3)
-		(layers "F.Cu" "B.Cu")
-		(net 0)
-	)
-	(via
 		(at 148.59 83.185)
-		(size 0.6)
-		(drill 0.3)
-		(layers "F.Cu" "B.Cu")
-		(net 0)
-	)
-	(via
-		(at 130.175 85.09)
 		(size 0.6)
 		(drill 0.3)
@@
 		(size 0.6)
 		(drill 0.3)
-		(layers "F.Cu" "B.Cu")
-		(net 0)
-	)
-	(via
-		(at 133.35 79.375)
-		(size 0.6)
-		(drill 0.3)
-		(layers "F.Cu" "B.Cu")
-		(net 0)
-	)
-	(via
-		(at 130.81 89.535)
-		(size 0.6)
-		(drill 0.3)

Commit message: Test commit 5
Routing:
- net (no net): vias 10 -> 16
Changed lines of the file:
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@@
+	)
+	(via
+		(at 133.35 85.09)
+		(size 0.6)
+		(drill 0.3)
+		(layers "F.Cu" "B.Cu")
+		(net 0)
 	)
 	(via
@@
 	)
 	(via
+		(at 138.43 82.55)
+		(size 0.6)
+		(drill 0.3)
+		(layers "F.Cu" "B.Cu")
+		(net 0)
+	)
+	(via
 		(at 153.67 88.265)
 		(size 0.6)
@@
 	)
 	(via
+		(at 130.81 86.36)
+		(size 0.6)
+		(drill 0.3)
+		(layers "F.Cu" "B.Cu")
+		(net 0)
+	)
+	(via
+		(at 138.43 90.17)
+		(size 0.6)
+		(drill 0.3)
+		(layers "F.Cu" "B.Cu")
+		(net 0)
+	)
+	(via
 		(at 148.59 83.185)
 		(size 0.6)
 		(drill 0.3)
+		(layers "F.Cu" "B.Cu")
+		(net 0)
+	)
+	(via
+		(at 131.445 90.805)
+		(size 0.6)
+		(drill 0.3)
+		(layers "F.Cu" "B.Cu")
+		(net 0)
+	)
+	(via
+		(at 137.795 85.725)
+		(size 0.6)
+		(drill 0.3)

Commit message: Testing commit 6
Routing:
- net (no net): vias 16 -> 13
Changed lines of the file:
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@@
-	)
-	(via
-		(at 146.685 75.565)
-		(size 0.6)
-		(drill 0.3)
-		(layers "F.Cu" "B.Cu")
-		(net 0)
-	)
-	(via
-		(at 153.035 76.2)
-		(size 0.6)
-		(drill 0.3)
-		(layers "F.Cu" "B.Cu")
-		(net 0)
 	)
 	(via
@@
 		(size 0.6)
 		(drill 0.3)
-		(layers "F.Cu" "B.Cu")
-		(net 0)
-	)
-	(via
-		(at 146.05 71.12)
-		(size 0.6)
-		(drill 0.3)
