File: testing/testing.kicad_pcb (KiCad board)
At the start: 2 copper layers, 45.8 x 63.6 mm, 0 parts

Commit message: Testing Commit 7 + Re-enabled things + Other minor naming things
Routing:
- net (no net): vias 13 -> 19
Changed lines of the file:
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@@
+	)
+	(via
+		(at 125.095 105.41)
+		(size 0.6)
+		(drill 0.3)
+		(layers "F.Cu" "B.Cu")
+		(net 0)
 	)
 	(via
@@
 	)
 	(via
+		(at 132.08 104.775)
+		(size 0.6)
+		(drill 0.3)
+		(layers "F.Cu" "B.Cu")
+		(net 0)
+	)
+	(via
 		(at 153.67 80.645)
 		(size 0.6)
@@
 	)
 	(via
+		(at 131.445 100.33)
+		(size 0.6)
+		(drill 0.3)
+		(layers "F.Cu" "B.Cu")
+		(net 0)
+	)
+	(via
 		(at 138.43 90.17)
+		(size 0.6)
+		(drill 0.3)
+		(layers "F.Cu" "B.Cu")
+		(net 0)
+	)
+	(via
+		(at 132.08 97.155)
 		(size 0.6)
 		(drill 0.3)
@@
 	)
 	(via
+		(at 124.46 100.965)
+		(size 0.6)
+		(drill 0.3)
+		(layers "F.Cu" "B.Cu")
+		(net 0)
+	)
+	(via
 		(at 137.795 85.725)
 		(size 0.6)
@@
 		(size 0.6)
 		(drill 0.3)
+		(layers "F.Cu" "B.Cu")
+		(net 0)
+	)
+	(via
+		(at 127 99.695)
+		(size 0.6)
+		(drill 0.3)

Commit message: Testing Commit 9
Changed lines of the file:
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@@
 	(net 0 "")
-	(gr_line
-		(start 159.0675 121.285)
-		(end 146.685 121.285)
-		(stroke
-			(width 0.2)
-			(type default)
-		)
-		(layer "F.Cu")
-	)
 	(gr_line
 		(start 135.255 112.395)
 		(end 156.21 116.84)
-		(stroke
-			(width 0.2)
-			(type default)
-		)
-		(layer "F.Cu")
-	)
-	(gr_line
-		(start 146.685 121.285)
-		(end 142.24 124.46)
-		(stroke
-			(width 0.2)
-			(type default)
-		)
-		(layer "F.Cu")
-	)
-	(gr_line
-		(start 154.305 96.52)
-		(end 146.05 93.345)
-		(stroke
-			(width 0.2)
-			(type default)
-		)
-		(layer "F.Cu")
-	)
-	(gr_line
-		(start 161.925 100.965)
-		(end 159.0675 121.285)
 		(stroke
 			(width 0.2)
@@
 		(stroke
 			(width 0.2)
-			(type default)
-		)
-		(layer "F.Cu")
-	)
-	(gr_line
-		(start 156.21 116.84)
-		(end 161.925 100.965)
-		(stroke
-			(width 0.2)
-			(type default)
-		)
-		(layer "F.Cu")
-	)
-	(gr_line
-		(start 142.24 124.46)
-		(end 154.305 96.52)
-		(stroke
-			(width 0.2)

Commit message: Testing Commit 12
Routing:
- net (no net): vias 19 -> 12
Changed lines of the file:
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@@
 	)
 	(net 0 "")
-	(gr_line
-		(start 135.255 112.395)
-		(end 156.21 116.84)
-		(stroke
-			(width 0.2)
-			(type default)
-		)
-		(layer "F.Cu")
-	)
-	(gr_line
-		(start 146.05 93.345)
-		(end 135.255 112.395)
-		(stroke
-			(width 0.2)
-			(type default)
-		)
-		(layer "F.Cu")
-	)
 	(gr_rect
 		(start 121.9 66.55)
@@
 	(via
 		(at 133.35 85.09)
-		(size 0.6)
-		(drill 0.3)
-		(layers "F.Cu" "B.Cu")
-		(net 0)
-	)
-	(via
-		(at 146.685 88.9)
-		(size 0.6)
-		(drill 0.3)
-		(layers "F.Cu" "B.Cu")
-		(net 0)
-	)
-	(via
-		(at 147.955 78.74)
 		(size 0.6)
 		(drill 0.3)
@@
 	)
 	(via
-		(at 153.67 88.265)
-		(size 0.6)
-		(drill 0.3)
-		(layers "F.Cu" "B.Cu")
-		(net 0)
-	)
-	(via
-		(at 153.035 83.82)
-		(size 0.6)
-		(drill 0.3)
-		(layers "F.Cu" "B.Cu")
-		(net 0)
-	)
-	(via
 		(at 132.08 104.775)
-		(size 0.6)
-		(drill 0.3)
-		(layers "F.Cu" "B.Cu")
-		(net 0)
-	)
-	(via
-		(at 153.67 80.645)
 		(size 0.6)
 		(drill 0.3)
@@
 	)
 	(via
-		(at 148.59 83.185)
-		(size 0.6)
-		(drill 0.3)
-		(layers "F.Cu" "B.Cu")
-		(net 0)
-	)
-	(via
 		(at 131.445 90.805)
 		(size 0.6)
@@
 		(size 0.6)
 		(drill 0.3)
-		(layers "F.Cu" "B.Cu")
-		(net 0)
-	)
-	(via
-		(at 146.05 84.455)
-		(size 0.6)
-		(drill 0.3)

Commit message: Test Commit 13
Routing:
- net (no net): vias 12 -> 20
Changed lines of the file:
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@@
+	)
+	(via
+		(at 146.05 96.52)
+		(size 0.6)
+		(drill 0.3)
+		(layers "F.Cu" "B.Cu")
+		(net 0)
 	)
 	(via
@@
 	)
 	(via
+		(at 141.605 95.885)
+		(size 0.6)
+		(drill 0.3)
+		(layers "F.Cu" "B.Cu")
+		(net 0)
+	)
+	(via
+		(at 139.7 111.125)
+		(size 0.6)
+		(drill 0.3)
+		(layers "F.Cu" "B.Cu")
+		(net 0)
+	)
+	(via
 		(at 132.08 104.775)
 		(size 0.6)
@@
 	)
 	(via
+		(at 146.685 100.965)
+		(size 0.6)
+		(drill 0.3)
+		(layers "F.Cu" "B.Cu")
+		(net 0)
+	)
+	(via
 		(at 130.81 86.36)
+		(size 0.6)
+		(drill 0.3)
+		(layers "F.Cu" "B.Cu")
+		(net 0)
+	)
+	(via
+		(at 139.7 101.6)
 		(size 0.6)
 		(drill 0.3)
@@
 	)
 	(via
+		(at 140.335 107.95)
+		(size 0.6)
+		(drill 0.3)
+		(layers "F.Cu" "B.Cu")
+		(net 0)
+	)
+	(via
 		(at 127 99.695)
 		(size 0.6)
 		(drill 0.3)
+		(layers "F.Cu" "B.Cu")
+		(net 0)
+	)
+	(via
+		(at 139.065 97.155)
+		(size 0.6)
+		(drill 0.3)
+		(layers "F.Cu" "B.Cu")
+		(net 0)
+	)
+	(via
+		(at 140.335 115.57)
+		(size 0.6)
+		(drill 0.3)
